Commit message: Place pendulum fixture mass on revolute link; relax RRBot e2e abs tolerance
The serial-chain model reads inertials only from revolute-joint child links,
so DrakePendulum_1DoF carries its full 1.0 kg on `arm` with a massless
`arm_com` marker, matching PyBullet inverse dynamics at tolerance 1e-4.
The RRBot end-to-end tolerance_abs=1e-2 absorbs its 1e-5 kg welded sensor links.

File: tests/assets/DrakePendulum_1DoF.urdf (robot description, URDF)
Before this commit: robot Pendulum, 4 links, 3 joints
Links:
- link arm: mass 0.5 -> 1.0
- link arm_com: mass 0.5 -> 0.0
